File: WM_RB-HAT.kicad_sch (KiCad schematic)
At the start: 98 parts, among them J1 Line R, J2 Output Stereo, J3 2x20 Pins, J5 Output Mono, J7 Line L, Q1 BC817, Q2 BFS17A, U1 WM8960, U3 74AHC1G14, U4 MCP1711T-33 /OT, X1 XO32, Y1 24MHz

Commit message: Added some notes for the next revision. General cleanup.
Parts:
- Logo1: now fitted
Other:
- note added: "Notas para correciones en REV-02: - Crosstalk @-60dB entre inputs J1 y J7 cuando.. . Reemplazar por jacks más chicos o alejar componentes para REV-02 - Ring y tips puenteado: puentea tip y sleeve en cables mono. Cortar pin ring en jack inputs como solución temporal."
- title: Raspberry Pi HAT -> Raspberry Audio Hat 
- moved on the sheet: FM1, FM2, FM3, H1, H2, H5, H6
